File: Battery Monitor/Battery Monitor v0.1/Battery Monitor v0.1.kicad_sch (KiCad schematic)
At the start: 55 parts, among them J1 XT60 M (Vertical), J10 Screw Terminal 5P, J11 Screw Terminal 5P, J12 Screw Terminal 5P, J13 JST-SH 3P, J14 JST-SH 3P, J15 JST-SH 3P, J16 JST-SH 3P, J17 JST-SH 3P, J18 JST-SH 3P, J2 Raspberry Pi 5, J3 2.54mm 3P, J4 2.54mm 3P, J5 2.54mm 3P, J6 2.54mm 3P, J7 Screw Terminal 5P, J8 Screw Terminal 5P, J9 Screw Terminal 5P, Q1 SUD50P10-43L, U1 15V~40V -> 12V 30A, U2 3.2~32V -> 5.1V 5A

Commit message: Finished schematic, added purchase links, began PCB layout
Parts:
- removed D5: LED, LED_SMD:LED_0805_2012Metric_Pad1.15x1.40mm_HandSolder, symbol Device:LED
- removed R2: 1k 0805, Resistor_SMD:R_0805_2012Metric_Pad1.20x1.40mm_HandSolder, symbol Device:R
- added C2: 1000u 50V (E), Capacitor_THT:CP_Radial_D13.0mm_P5.00mm, symbol Device:C_Polarized
- added C3: 0.1u 50V 1206 (C), Capacitor_SMD:C_1206_3216Metric_Pad1.33x1.80mm_HandSolder, symbol Device:C
- added D7: Green 0805, LED_SMD:LED_0805_2012Metric_Pad1.15x1.40mm_HandSolder, symbol Device:LED
- added FB3: BLM21PG220, Inductor_SMD:L_0805_2012Metric_Pad1.05x1.20mm_HandSolder, symbol Device:FerriteBead
- added R4, R7: 470R 0805, Resistor_SMD:R_0805_2012Metric_Pad1.20x1.40mm_HandSolder, symbol Device:R
- added U2: 12V~24V -> 7.5V 5A, Library:Buck_Converter_44x24.5mm_1, symbol Generic_Buck_Converter:Generic Buck Converter
- A1: value RaspberryPi_Pico -> RaspberryPi Pico; Taobao (none) -> https://item.taobao.com/item.htm?id=643838129251&spm=a312a.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; now left out of the parts list
- C1: value 2200u 50V (E) -> 1000u 50V (E); footprint Capacitor_THT:CP_Radial_D16.0mm_P7.50mm -> Capacitor_THT:CP_Radial_D13.0mm_P5.00mm; Taobao (none) -> https://item.taobao.com/item.htm?id=522579424493&spm=a312a.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
- C10: renamed from C3; footprint Capacitor_THT:CP_Radial_D16.0mm_P7.50mm -> Capacitor_THT:CP_Radial_D8.0mm_P3.50mm; Taobao (none) -> https://item.taobao.com/item.htm?id=564996742055&skuId=5731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
- C11: renamed from C7; footprint Capacitor_THT:CP_Radial_D16.0mm_P7.50mm -> Capacitor_THT:CP_Radial_D8.0mm_P3.50mm; Taobao (none) -> https://item.taobao.com/item.htm?id=564996742055&skuId=5731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
- C4: renamed from C9; value 100nF -> 0.1u 50V 1206 (C); Taobao (none) -> https://item.taobao.com/item.htm?id=522554243102&spm=a312a.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
- C5: renamed from C4; Taobao (none) -> https://item.taobao.com/item.htm?id=565000050337&spm=a312a.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
- C6: renamed from C5; value 100u 25V (T) -> 100u 50V (E); footprint Capacitor_SMD:C_1206_3216Metric_Pad1.33x1.80mm_HandSolder -> Capacitor_THT:CP_Radial_D8.0mm_P3.50mm; Taobao (none) -> https://item.taobao.com/item.htm?id=564996742055&skuId=5731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
- C7: renamed from C6; value 0.1uF (C) -> 0.1u 50V 1206 (C); Taobao (none) -> https://item.taobao.com/item.htm?id=522554243102&spm=a312a.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
- C8: renamed from C2; footprint Capacitor_THT:CP_Radial_D16.0mm_P7.50mm -> Capacitor_THT:CP_Radial_D8.0mm_P3.50mm; Taobao (none) -> https://item.taobao.com/item.htm?id=564996742055&skuId=5731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
- C9: renamed from C8; footprint Capacitor_THT:CP_Radial_D16.0mm_P7.50mm -> Capacitor_THT:CP_Radial_D8.0mm_P3.50mm; Taobao (none) -> https://item.taobao.com/item.htm?id=564996742055&skuId=5731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
- D1: value 15V -> 14.7V; Taobao (none) -> https://item.taobao.com/item.htm?abbucket=6&id=695101953366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
- D2: renamed from D6; value 3V3 -> 3.3V; Taobao (none) -> https://item.taobao.com/item.htm?abbucket=6&id=697021351088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
- D3: renamed from D7; Taobao (none) -> https://item.taobao.com/item.htm?id=661190438436&spm=a312a.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
- D4: renamed from D8; value SMAJ5.0A -> SMAJ6.0A; Taobao (none) -> https://item.taobao.com/item.htm?id=626801460817&spm=a312a.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
- D5: renamed from D2; value LED -> Green 0805; Taobao (none) -> https://item.taobao.com/item.htm?id=522554271548&spm=a312a.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
- D6: renamed from D3; value LED -> Green 0805; Taobao (none) -> https://item.taobao.com/item.htm?id=522554271548&spm=a312a.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
- D8: renamed from D4; value LED -> Green 0805; Taobao (none) -> https://item.taobao.com/item.htm?id=522554271548&spm=a312a.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
- F1: Taobao (none) -> https://item.taobao.com/item.htm?id=646550973988&mi_id=0000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
- F2: value 5A Polyfuse -> 5A 1812; Taobao (none) -> https://detail.tmall.com/item.htm?id=680110340340&mi_id=000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
- F3: value 500mA Polyfuse -> 500mA 1206; Taobao (none) -> https://detail.tmall.com/item.htm?id=671048655631&mi_id=000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
- FB1, FB2: Taobao (none) -> https://detail.tmall.com/item.htm?abbucket=6&id=73393430147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
- H1, H2, H3, H4: value 3.2mm M3 -> M3 3.2mm; footprint MountingHole:MountingHole_3.2mm_M3_DIN965_Pad_TopBottom -> MountingHole:MountingHole_3.2mm_M3_DIN965_Pad
- J1: Taobao (none) -> https://item.taobao.com/item.htm?id=599294573848&skuId=4184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
- J10: renamed from J6; footprint (none) -> Connector_PinHeader_2.54mm:PinHeader_1x03_P2.54mm_Vertical; Taobao (none) -> https://item.taobao.com/item.htm?id=522579376259&skuId=6139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
- J11: renamed from J4; footprint (none) -> Connector_PinHeader_2.54mm:PinHeader_1x03_P2.54mm_Vertical; Taobao (none) -> https://item.taobao.com/item.htm?id=522579376259&skuId=6139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
- J12: renamed from J5; footprint (none) -> Connector_PinHeader_2.54mm:PinHeader_1x03_P2.54mm_Vertical; Taobao (none) -> https://item.taobao.com/item.htm?id=522579376259&skuId=6139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
- J13, J14, J15, J16, J17, J18: footprint (none) -> Connector_JST:JST_SH_BM03B-SRSS-TB_1x03-1MP_P1.00mm_Vertical; Taobao (none) -> https://item.taobao.com/item.htm?abbucket=6&id=616913039189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
- J2: footprint Connector_PinSocket_2.54mm:PinSocket_2x20_P2.54mm_Vertical -> Library:Raspberry_Pi_5; Taobao (none) -> https://item.taobao.com/item.htm?id=522576768218&skuId=3150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
- J3: renamed from J7; value Screw Terminal 5P -> Screw 2.54mm 5P; footprint (none) -> Connector_PinHeader_2.54mm:PinHeader_1x05_P2.54mm_Vertical; Taobao (none) -> https://item.taobao.com/item.htm?id=642057328277&skuId=4619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
- J4: renamed from J8; footprint (none) -> Connector_PinHeader_2.54mm:PinHeader_1x05_P2.54mm_Vertical; Taobao (none) -> https://item.taobao.com/item.htm?id=642057328277&skuId=4619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
- J5: renamed from J9; footprint (none) -> Connector_PinHeader_2.54mm:PinHeader_1x05_P2.54mm_Vertical; Taobao (none) -> https://item.taobao.com/item.htm?id=642057328277&skuId=4619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
- J6: renamed from J10; footprint (none) -> Connector_PinHeader_2.54mm:PinHeader_1x05_P2.54mm_Vertical; Taobao (none) -> https://item.taobao.com/item.htm?id=642057328277&skuId=4619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
- J7: renamed from J11; footprint (none) -> Connector_PinHeader_2.54mm:PinHeader_1x05_P2.54mm_Vertical; Taobao (none) -> https://item.taobao.com/item.htm?id=642057328277&skuId=4619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
- J8: renamed from J12; footprint (none) -> Connector_PinHeader_2.54mm:PinHeader_1x05_P2.54mm_Vertical; Taobao (none) -> https://item.taobao.com/item.htm?id=642057328277&skuId=4619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
- J9: renamed from J3; footprint (none) -> Connector_PinHeader_2.54mm:PinHeader_1x03_P2.54mm_Vertical; Taobao (none) -> https://item.taobao.com/item.htm?id=522579376259&skuId=6139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
- Q1: value SUD50P10-43L -> NCE1540KA; Taobao (none) -> https://item.taobao.com/item.htm?id=809752933171&spm=a312a.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
- R1: value 100k 0805 -> 100k 0805 1%; Taobao (none) -> https://item.taobao.com/item.htm?abbucket=6&id=526088038633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
- R2: renamed from R6; Taobao (none) -> https://item.taobao.com/item.htm?abbucket=6&id=526088038633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
- R3: renamed from R7; value 13.7k -> 13.3k 0805 1%; Taobao (none) -> https://item.taobao.com/item.htm?abbucket=6&id=526088038633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
- R5: value 50R -> 470R 0805; Taobao (none) -> https://item.taobao.com/item.htm?id=522573121620&skuId=5702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
- R6: renamed from R3; value 480R -> 470R 0805; Taobao (none) -> https://item.taobao.com/item.htm?id=522573121620&skuId=5702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
- R8: renamed from R4; value 150R -> 470R 0805; Taobao (none) -> https://item.taobao.com/item.htm?id=522573121620&skuId=5702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
- U1: Taobao (none) -> https://item.taobao.com/item.htm?id=535067252604&last_time=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
- U3: renamed from U2; Taobao (none) -> https://item.taobao.com/item.htm?id=530479908999&spm=a312a.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
Connections:
- net +12V: now also J3.5 (Pin_5), J4.5 (Pin_5), J5.5 (Pin_5), J6.5 (Pin_5), J7.5 (Pin_5), J8.5 (Pin_5); no longer C10.1, C11.1, C8.1, C9.1, J10.2 (Pin_2), J11.2 (Pin_2), J12.2 (Pin_2), J13.2 (Pin_2), J14.2 (Pin_2), J15.2 (Pin_2), J16.2 (Pin_2), J17.2 (Pin_2), J18.2 (Pin_2), J3.1 (Pin_1), J4.1 (Pin_1), J5.1 (Pin_1), J6.1 (Pin_1), J7.1 (Pin_1), J8.1 (Pin_1), J9.2 (Pin_2)
- net +3V3: now also A1.36 (3V3), FB3.2
- net +5.1V: now also J13.2 (Pin_2), J14.2 (Pin_2), J15.2 (Pin_2), J16.2 (Pin_2), J17.2 (Pin_2), J18.2 (Pin_2)
- net +BATT: now also C2.1, U2.4 (VIN+)
- net BLDC_0: now also A1.4 (GPIO2); no longer A1.9 (GPIO6)
- net BLDC_1: now also A1.5 (GPIO3); no longer A1.10 (GPIO7)
- net BLDC_2: now also A1.6 (GPIO4); no longer A1.11 (GPIO8)
- net BLDC_3: now also A1.7 (GPIO5); no longer A1.12 (GPIO9)
- net BLDC_4: now also A1.9 (GPIO6); no longer A1.14 (GPIO10)
- net BLDC_5: now also A1.10 (GPIO7); no longer A1.15 (GPIO11)
- net GND: now also J10.1 (Pin_1), J11.1 (Pin_1), J12.1 (Pin_1), J3.1 (Pin_1), J4.1 (Pin_1), J5.1 (Pin_1), J6.1 (Pin_1), J7.1 (Pin_1), J8.1 (Pin_1), J9.1 (Pin_1), C2.2, C3.2, R7.1, U2.2 (-VDC), U2.3 (VIN-); no longer J10.3 (Pin_3), J11.3 (Pin_3), J12.3 (Pin_3), J3.5 (Pin_5), J4.5 (Pin_5), J5.5 (Pin_5), J6.5 (Pin_5), J7.5 (Pin_5), J8.5 (Pin_5), J9.3 (Pin_3)
- net SERVO_0: now also A1.11 (GPIO8), J9.3 (Pin_3); no longer A1.4 (GPIO2), J9.1 (Pin_1)
- net SERVO_1: now also A1.12 (GPIO9), J10.3 (Pin_3); no longer A1.5 (GPIO3), J10.1 (Pin_1)
- net SERVO_2: now also A1.14 (GPIO10), J11.3 (Pin_3); no longer A1.6 (GPIO4), J11.1 (Pin_1)
- net SERVO_3: now also A1.15 (GPIO11), J12.3 (Pin_3); no longer A1.7 (GPIO5), J12.1 (Pin_1)
- net at R5.2: now also R4.1
- net at A1.35 (ADC_VREF): now also C3.1, FB3.1
- net at D5.1 (K): now also R4.2
- new net: D7.1 (K), R7.2
- new net +7.5V: C10.1, C11.1, C8.1, C9.1, D7.2 (A), J10.2 (Pin_2), J11.2 (Pin_2), J12.2 (Pin_2), J9.2 (Pin_2), U2.1 (+VDC)
- no-connect marks 48 -> 46
Other:
- title: Prototype Rover Battery Monitor v0.1 -> Prototype Rover PCB v0.1
- moved on the sheet: A1, C1, C10, C11, C4, C5, C6, C7, C8, C9, D1, D2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
