File: PCB v0.2.kicad_sch (KiCad schematic)
At the start: 59 parts, among them J1 XT60 M (Vertical), J10 2.54mm 3P, J11 2.54mm 3P, J12 2.54mm 3P, J13 JST-SH 3P, J14 JST-SH 3P, J15 JST-SH 3P, J16 JST-SH 3P, J17 JST-SH 3P, J18 JST-SH 3P, J2 Raspberry Pi 5, J3 Screw 2.54mm 5P, J4 Screw Terminal 5P, J5 Screw Terminal 5P, J6 Screw Terminal 5P, J7 Screw Terminal 5P, J8 Screw Terminal 5P, J9 2.54mm 3P, Q1 NCE1540KA, U1 15V~40V -> 12V 30A, U1 3.2~32V -> 5.1V 5A, U2 12V~24V -> 7.5V 5A

Commit message: Replaced DC/DC symbol in schematic with appropriate XT30 connectors, fixed XT60 polarity
Parts:
- removed J1: XT60 M (Vertical), Connector_AMASS:AMASS_XT60PW-M_1x02_P7.20mm_Horizontal, symbol Connector_Generic:Conn_01x02
- removed U1: 15V~40V -> 12V 30A, Library:Buck_Converter_74x74mm, symbol Generic_Buck_Converter:Generic Buck Converter
- removed U2: 12V~24V -> 7.5V 5A, Library:Buck_Converter_44x24.5mm_1, symbol Generic_Buck_Converter:Generic Buck Converter
- added J1: XT60-M, Connector_AMASS:AMASS_XT60PW-M_1x02_P7.20mm_Horizontal, symbol Connector_Generic_MountingPin:Conn_01x02_MountingPin
- added J3, J5: XT30-F, Connector_AMASS:AMASS_XT30PW-F_1x02_P2.50mm_Horizontal, symbol Connector_Generic_MountingPin:Conn_01x02_MountingPin
- added J4, J6: XT30-M, Connector_AMASS:AMASS_XT30PW-M_1x02_P2.50mm_Horizontal, symbol Connector_Generic_MountingPin:Conn_01x02_MountingPin
- J10: renamed from J6; value Screw Terminal 5P -> Screw 2.54mm 5P
- J11: renamed from J7; value Screw Terminal 5P -> Screw 2.54mm 5P
- J12: renamed from J8; value Screw Terminal 5P -> Screw 2.54mm 5P
- J8: renamed from J4; value Screw Terminal 5P -> Screw 2.54mm 5P
- J9: renamed from J5; value Screw Terminal 5P -> Screw 2.54mm 5P
- renumbered J9 to J13, J10 to J14, J11 to J15, J12 to J16, J13 to J17, J14 to J18, J15 to J19, J16 to J20, J17 to J21, J18 to J22, J3 to J7
Connections:
- net +12V: now also J4.2 (Pin_2)
- net +7.5V: now also J6.2 (Pin_2)
- net +BATT: now also J3.2 (Pin_2), J5.2 (Pin_2)
- net GND: now also J1.1 (Pin_1), J1.MP (MountPin), J3.1 (Pin_1), J3.MP (MountPin), J4.1 (Pin_1), J4.MP (MountPin), J5.1 (Pin_1), J5.MP (MountPin), J6.1 (Pin_1), J6.MP (MountPin)
- net at F1.1: now also J1.2 (Pin_2)
Other:
- note added: "External DC/DC Converter"
- moved on the sheet: J17, J18, J19, J20, J21, J22
