File: PCB v0.2.kicad_sch (KiCad schematic)
At the start: 67 parts, among them J1 XT60-M, J10 Screw 2.54mm 5P, J11 Screw 2.54mm 5P, J12 Screw 2.54mm 5P, J13 2.54mm 3P, J14 2.54mm 3P, J15 2.54mm 3P, J16 2.54mm 3P, J17 JST-SH 3P, J18 JST-SH 3P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

Commit message: Preparing for v0.3
Parts:
- J2: footprint Library:Raspberry_Pi_5 -> Library:raspberrypi_2_3
- Q1: value NCE1540KA -> NCE15P25JK
Changed lines of the file:
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@@
 			)
 		)
-		(property "Footprint" "Library:Raspberry_Pi_5"
+		(property "Footprint" "Library:raspberrypi_2_3"
 			(at 294.894 114.808 0)
 			(hide yes)
@@
 			)
 		)
-		(property "Value" "NCE1540KA"
+		(property "Value" "NCE15P25JK"
 			(at 80.01 33.02 90)
 			(show_name no)
