File: PCB v0.2.kicad_pcb (KiCad board)
At the start: 2 copper layers, 94.7 x 96.8 mm, 67 parts, among them J1 XT60-M, J10 Screw 2.54mm 5P, J11 Screw 2.54mm 5P, J12 Screw 2.54mm 5P, J13 2.54mm 3P, J14 2.54mm 3P, J15 2.54mm 3P, J16 2.54mm 3P, J17 JST-SH 3P, J18 JST-SH 3P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

Commit message: Preparing for v0.3
Parts:
- J2: footprint Library:Raspberry_Pi_5 -> Library:raspberrypi_2_3
- Q1: value NCE1540KA -> NCE15P25JK
- moved C6 262.5 mm to (-83.6, 112.5), turned to 0 degrees
- moved J20 258.2 mm to (-73.1, 129.6)
- moved J21 257.2 mm to (-73.1, 135.9)
- moved J22 256.2 mm to (-73.1, 142.1)
- moved J17 230.7 mm to (-73.1, 110.9)
- moved J18 229.9 mm to (-73.1, 117.1)
- moved J19 229.1 mm to (-73.1, 123.4)
- moved C8 226.2 mm to (-83.6, 122.1), turned to 0 degrees
- moved C9 225.9 mm to (-83.6, 131.6), turned to 0 degrees
- moved C10 225.6 mm to (-83.6, 141.2), turned to 0 degrees
- moved C11 225.3 mm to (-83.6, 150.7), turned to 0 degrees
- moved D8 224.8 mm to (-36.1, 155.3), turned to 0 degrees
- moved C7 223.8 mm to (-42.2, 150.9), turned to 0 degrees
- moved C3 223.7 mm to (-42.2, 144.2)
- moved C4 223.0 mm to (-42.2, 147.5)
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Routing:
- net +BATT: track 167.0 -> 0.00 mm, vias 1 -> 0
- net +5.1V: track 101.1 -> 0.00 mm, vias 1 -> 0
- net +7.5V: track 99.9 -> 0.00 mm, vias 2 -> 0
- net /REV_5: track 84.1 -> 0.00 mm, vias 1 -> 0
- net /BLDC_5: track 80.4 -> 0.00 mm, vias 1 -> 0
- net /ENC_0: track 79.6 -> 0.00 mm
- net /ENC_3: track 73.6 -> 0.00 mm
- net /ENC_1: track 72.4 -> 0.00 mm
- net /ENC_2: track 65.9 -> 0.00 mm
- net /REV_3: track 60.5 -> 0.00 mm, vias 1 -> 0
- net /BLDC_3: track 59.8 -> 0.00 mm, vias 1 -> 0
- net /REV_1: track 58.8 -> 0.00 mm, vias 1 -> 0
- net /BLDC_1: track 56.8 -> 0.00 mm, vias 1 -> 0
- net /REV_2: track 52.3 -> 0.00 mm, vias 1 -> 0
- net /BLDC_4: track 52.1 -> 0.00 mm, vias 1 -> 0
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- removed copper zone on F.Cu, net +5.1V
- removed copper zone on F.Cu, net +7.5V
- removed copper zone on F.Cu, net +BATT
- removed copper zone on B.Cu, net GND
- removed copper zone on F.Cu, net GND
- removed copper zone on B.Cu, net Net-(FB1-Pad1)
- removed copper zone on F.Cu, net Net-(FB1-Pad1)
- removed copper zone on B.Cu, net Net-(J1-Pin_2)
- removed copper zone on F.Cu, net Net-(J1-Pin_2)
- removed copper zone on B.Cu, net Net-(Q1-D)
- removed copper zone on F.Cu, net Net-(Q1-D)
Other:
- board size 94.7 x 96.8 mm -> 102.5 x 102.5 mm
- board text removed: "0"
- board text removed: "1"
- board text removed: "12V"
- board text removed: "12V IN →"
- board text removed: "2"
- board text removed: "22.2V"
- board text removed: "3"
- board text removed: "4"
- board text removed: "5"
- board text removed: "5.1V"
- board text removed: "7.5V"
- board text removed: "7.5V IN →"
- board text removed: "BATTERY IN →"
- board text removed: "C8-11"
- board text removed: "D5-8"
- board text removed: "DC MOTORS"
- board text removed: "Designed by: Ilo Japar"
- board text removed: "ENCODERS"
- board text removed: "HKU MARTIANS"
- board text removed: "J13-18"
- board text removed: "J3-8"
- board text removed: "J9-12"
- board text removed: "POWER"
- board text removed: "Prototype Rover PCB v0.2 rev B"
- board text removed: "R4-8"
- board text removed: "SERVOS"
